File: kicad/temp.kicad_pcb (KiCad board)
At the start: 2 copper layers, 10 parts, among them J1 Conn_01x06_Male, J2 Conn_01x02_Female, M1 Motor_DC, Q1 IRF540N, U1 LM7805_TO220, U2 PIC16F684-IP

Commit message: kicad
Parts:
- added J10: Conn_01x01_Female, Connector_PinHeader_2.54mm:PinHeader_1x01_P2.54mm_Vertical, F.Cu at (125.7, 104.8)
- added J11: Conn_01x01_Female, Connector_PinHeader_2.54mm:PinHeader_1x01_P2.54mm_Vertical, F.Cu at (125.7, 108.6)
- added J12: Conn_01x01_Female, Connector_PinHeader_2.54mm:PinHeader_1x01_P2.54mm_Vertical, F.Cu at (159.4, 108.6)
- added J13: Conn_01x01_Female, Connector_PinHeader_2.54mm:PinHeader_1x01_P2.54mm_Vertical, F.Cu at (159.4, 104.8)
- added J14: Conn_01x01_Female, Connector_PinHeader_2.54mm:PinHeader_1x01_P2.54mm_Vertical, F.Cu at (159.4, 101.0)
- added J15: Conn_01x01_Female, Connector_PinHeader_2.54mm:PinHeader_1x01_P2.54mm_Vertical, F.Cu at (125.7, 85.7)
- added J16: Conn_01x01_Female, Connector_PinHeader_2.54mm:PinHeader_1x01_P2.54mm_Vertical, F.Cu at (159.4, 85.7)
- added J3: Conn_01x01_Female, Connector_PinHeader_2.54mm:PinHeader_1x01_P2.54mm_Vertical, F.Cu at (159.4, 89.5)
- added J4: Conn_01x01_Female, Connector_PinHeader_2.54mm:PinHeader_1x01_P2.54mm_Vertical, F.Cu at (159.4, 93.3)
- added J5: Conn_01x01_Female, Connector_PinHeader_2.54mm:PinHeader_1x01_P2.54mm_Vertical, F.Cu at (159.4, 97.2)
- added J6: Conn_01x01_Female, Connector_PinHeader_2.54mm:PinHeader_1x01_P2.54mm_Vertical, F.Cu at (125.7, 97.2)
- added J7: Conn_01x01_Female, Connector_PinHeader_2.54mm:PinHeader_1x01_P2.54mm_Vertical, F.Cu at (125.7, 93.3)
- added J8: Conn_01x01_Female, Connector_PinHeader_2.54mm:PinHeader_1x01_P2.54mm_Vertical, F.Cu at (125.7, 89.5)
- added J9: Conn_01x01_Female, Connector_PinHeader_2.54mm:PinHeader_1x01_P2.54mm_Vertical, F.Cu at (125.7, 101.0)
- moved J2 71.7 mm to (141.0, 51.4), turned to 90 degrees
- moved C1 51.6 mm to (150.5, 67.3), turned to 180 degrees
- moved M1 50.4 mm to (146.1, 138.4), turned to 90 degrees
- moved D1 49.0 mm to (144.1, 127.6)
- moved Q1 41.7 mm to (136.5, 139.7), turned to 90 degrees
- moved C3 40.1 mm to (134.0, 67.3), turned to 0 degrees
- moved U1 27.3 mm to (144.8, 59.1), turned to 180 degrees
- moved R1 21.3 mm to (130.8, 127.6)
- moved U2 13.5 mm to (139.1, 90.8)
- moved J1 11.1 mm to (136.5, 79.4)
Connections:
- net Net-(Q1-Pad1) renamed Ben5
- J1 pad 5: Net-(J1-Pad5) -> PGC
- U2 pad 10: Net-(U2-Pad10) -> Ben10
- U2 pad 11: Net-(U2-Pad11) -> Ben11
- U2 pad 2: Net-(U2-Pad2) -> Ben2
- U2 pad 3: Net-(U2-Pad3) -> Ben3
- U2 pad 6: Net-(U2-Pad6) -> Ben6
- U2 pad 7: Net-(U2-Pad7) -> Ben7
- U2 pad 8: Net-(U2-Pad8) -> Ben8
- U2 pad 9: Net-(U2-Pad9) -> Ben9
Routing:
- net Earth: track 0.00 -> 120.0 mm
- net VCC: track 0.00 -> 113.1 mm, vias 0 -> 1
- net Ben5: track 0.00 -> 61.2 mm
- net 5V: track 0.00 -> 59.0 mm
- net PGC: track 0.00 -> 53.6 mm
- net Vpp: track 0.00 -> 46.9 mm
- net PGD: track 0.00 -> 46.8 mm
- net Net-(D1-Pad2): track 0.00 -> 33.2 mm, vias 0 -> 1
- net Ben2: track 0.00 -> 15.8 mm
- net Ben3: track 0.00 -> 14.4 mm
- net Ben7: track 0.00 -> 14.4 mm
- net Ben6: track 0.00 -> 13.9 mm
- net Ben8: track 0.00 -> 13.8 mm
- net Ben9: track 0.00 -> 13.2 mm
- net Ben11: track 0.00 -> 13.2 mm
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- added copper zone on B.Cu, net Earth
